File: Hardware/ShortWaveModule_SmallBoard.sch (EAGLE design)
At the start: 54 parts, among them J1 CONN_42.54_SCREW, J2 CONN_42.54, J3 CONN_42.54, J4 CONN_42.54, Q1 2N7002, Q2 2N7002, Q3 DMG3404

Commit message: Added pullups to shortwave module
Added pullups to onboard I2C on shortwave module, still need to fix silk screen and update parts before ready to ship
Parts:
- added R3, R4: 10k, bschulz_passives:R-EU_10KR0603
- U$11, U$12: value LTC2054HV -> LTC2050; device bschulz:LTC2054HV -> bschulz:LTC2050
Connections:
- net 3V3: now also R3.2, R4.2
- net SCL: now also R3.1
- net SDA: now also R4.1
Changed lines of the file:
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@@
 <part name="U$9" library="bschulz" deviceset="PHOTODIODE" device="VEMD1060" value="PHOTODIODEVEMD1060"/>
 <part name="U$10" library="bschulz" deviceset="PHOTODIODE" device="SD003-151-001"/>
-<part name="U$11" library="bschulz" deviceset="LTC2054" device="" technology="HV"/>
-<part name="U$12" library="bschulz" deviceset="LTC2054" device="" technology="HV"/>
+<part name="U$11" library="bschulz" deviceset="LTC2050" device="" value="LTC2050"/>
+<part name="U$12" library="bschulz" deviceset="LTC2050" device="" value="LTC2050"/>
 <part name="R15" library="bschulz_passives" deviceset="R-EU_" device="R0603" value="1k"/>
 <part name="C13" library="bschulz_passives" deviceset="C-EU" device="C0603" value="0.15uF"/>
@@
 <part name="JP2" library="SparkFun-Jumpers" library_urn="urn:adsk.eagle:library:528" deviceset="JUMPER-SMT_2_NO" device="_SILK" package3d_urn="urn:adsk.eagle:package:39279/1"/>
 <part name="R2" library="bschulz_passives" deviceset="R-EU_" device="R0603" technology="10K" value="10k"/>
+<part name="R3" library="bschulz_passives" deviceset="R-EU_" device="R0603" technology="10K" value="10k"/>
+<part name="R4" library="bschulz_passives" deviceset="R-EU_" device="R0603" technology="10K" value="10k"/>
 </parts>
 <sheets>
@@
 </instance>
 <instance part="R2" gate="G$1" x="71.12" y="175.26" rot="R180"/>
+<instance part="R3" gate="G$1" x="60.96" y="121.92" rot="R90"/>
+<instance part="R4" gate="G$1" x="76.2" y="121.92" rot="R90"/>
 </instances>
 <busses>
@@
 <wire x1="76.2" y1="175.26" x2="81.28" y2="175.26" width="0.1524" layer="91"/>
 <label x="78.74" y="175.26" size="1.778" layer="95" ratio="15"/>
+</segment>
+<segment>
+<pinref part="R4" gate="G$1" pin="2"/>
+<wire x1="76.2" y1="127" x2="76.2" y2="129.54" width="0.1524" layer="91"/>
+<wire x1="76.2" y1="129.54" x2="81.28" y2="129.54" width="0.1524" layer="91"/>
+<label x="76.2" y="129.54" size="1.778" layer="95"/>
+</segment>
+<segment>
+<pinref part="R3" gate="G$1" pin="2"/>
+<wire x1="60.96" y1="127" x2="60.96" y2="129.54" width="0.1524" layer="91"/>
+<wire x1="60.96" y1="129.54" x2="66.04" y2="129.54" width="0.1524" layer="91"/>
+<label x="60.96" y="129.54" size="1.778" layer="95"/>
 </segment>
 </net>
@@
 <label x="195.58" y="144.78" size="1.778" layer="95"/>
 </segment>
+<segment>
+<pinref part="R4" gate="G$1" pin="1"/>
+<wire x1="76.2" y1="116.84" x2="68.58" y2="116.84" width="0.1524" layer="91"/>
+<label x="66.04" y="116.84" size="1.778" layer="95"/>
+</segment>
 </net>
 <net name="SCL" class="0">
@@
 <label x="195.58" y="142.24" size="1.778" layer="95"/>
 </segment>
+<segment>
+<pinref part="R3" gate="G$1" pin="1"/>
+<wire x1="60.96" y1="116.84" x2="53.34" y2="116.84" width="0.1524" layer="91"/>
+<label x="50.8" y="116.84" size="1.778" layer="95"/>
+</segment>
 </net>

Commit message: Updated parts and BOM
Parts:
- removed C16: 1uF, bschulz_passives:C-EU1UFC0603
- removed C17: 0.1uF, bschulz_passives:C-EU0.1UFC0603
- removed H3: (no value), bschulz:MOUNTING_HOLE4_NP
- removed R19, R20: 1k, bschulz_passives:R-EU_R0603
- removed R21: 10k, bschulz_passives:R-EU_10KR0603
- removed RT2: (no value), bschulz:THERMISTOR10K
- added C12, C4: 0.1uF, bschulz_passives:C-EU0.1UFC0603
- added H2: (no value), bschulz:MOUNTING_HOLE4_NP
- added R5: 10k, bschulz_passives:R-EU_P10KR0603
- added R6, R7: 10k, bschulz_passives:R-EU_10KR0603
- added RT1: 10k, bschulz:THERMISTOR10K
- C1: value 0.1uF -> 10uF; device bschulz_passives:C-EU0.1UFC0603 -> bschulz_passives:C-EU10UFC0805
- C13: value 0.15uF -> 1uF; device bschulz_passives:C-EUC0603 -> bschulz_passives:C-EU1UFC0603
- C14: value 0.15uF -> 0.1uF; device bschulz_passives:C-EUC0603 -> bschulz_passives:C-EU0.1UFC0603
- C2: value 10uF -> 0.15uF; device bschulz_passives:C-EU10UFC0805 -> bschulz_passives:C-EU0.15UFC0603
- C3: value 0.1uF -> 0.15uF; device bschulz_passives:C-EU0.1UFC0603 -> bschulz_passives:C-EU0.15UFC0603
- C5: value 1uF -> 0.1uF; device bschulz_passives:C-EU1UFC0603 -> bschulz_passives:C-EU0.1UFC0603
- C7: value 0.1uF -> 1uF; device bschulz_passives:C-EU0.1UFC0603 -> bschulz_passives:C-EU1UFC0603
- R1: value 27R -> 1k; device bschulz:R-EU_27R0603 -> bschulz_passives:R-EU_P1KR0603
- R10, R2, R9: value 10k -> 1k; device bschulz_passives:R-EU_10KR0603 -> bschulz_passives:R-EU_P1KR0603
- R15: value 1k -> 10k; device bschulz_passives:R-EU_R0603 -> bschulz_passives:R-EU_10KR0603
- R16: value 47k -> 10k; device bschulz_passives:R-EU_R0603 -> bschulz_passives:R-EU_10KR0603
- R17: value 1k -> 10k; device bschulz_passives:R-EU_R0603 -> bschulz_passives:R-EU_P10KR0603; DIGIKEY (none) -> P10KDBCT-ND; MF (none) -> Panasonic; MPN (none) -> ERA-3AEB103V
- R18: value 1M -> 10k; device bschulz_passives:R-EU_R0603 -> bschulz_passives:R-EU_10KR0603
- R3: value 10k -> 27R; device bschulz_passives:R-EU_10KR0603 -> bschulz:R-EU_27R0603
- R4: value 10k -> 100k; device bschulz_passives:R-EU_10KR0603 -> bschulz_passives:R-EU_P100KR0603
- renumbered ADS1115 to U5, C18 to C11, U$1 to U2, U$10 to D1, U$11 to U3, U$12 to U4, U$2 to U7, U$3 to U8, U$4 to U1, U$5 to U6, U$9 to D2
Connections:
- net !ADC_INT: now also R18.1; no longer R13.1
- net !LUX_INT: now also R14.1; no longer R12.1
- net !RESET: now also R11.1; no longer R14.1
- net 3V3: now also C12.1, C14.1, C15.1, C4.1, C5.1, R11.2, R18.2, R3.1, R6.2, R7.1, RT1.2; no longer C17.1, C2.1, C6.1, C7.1, C8.1, R1.1, R10.2, R2.1, R21.2, R3.2, R4.2
- net AOUT_MWAVE: now also C6.1, R9.2; no longer C16.1, R19.2
- net AOUT_SWAVE: now also C7.1, R10.2; no longer C15.1, R20.2
- net AOUT_THERM: now also C8.1, R17.2, RT1.1; no longer C3.1, R21.1, RT2.1
- net GND: now also C12.2, C13.2, C14.2, C4.2, R17.1; no longer C16.2, C17.2, C2.2, C3.2, RT2.2
- net N$1: now also R7.2; no longer R2.2
- net N$10: now also R1.1, R4.1; no longer R17.1, R18.1
- net N$11: now also C2.1, R1.2; no longer C14.1, R17.2
- net N$12: now also C2.2, R4.2, R9.1; no longer C14.2, R18.2, R19.1
- net N$13: now also C3.2, R10.1, R5.2; no longer C13.2, R16.2, R20.1
- net N$8: now also C3.1, R2.2; no longer C13.1, R15.2
- net N$9: now also R2.1, R5.1; no longer R15.1, R16.1
- net SCL: now also R6.1; no longer R3.1
- net SCL_EXT: now also R13.1; no longer R10.1
- net SCL_EXT_HV: now also R16.1; no longer R11.1
- net SDA: now also R8.1; no longer R4.1
- net SDA_EXT: now also R12.1; no longer R8.1
- net SDA_EXT_HV: now also R15.1; no longer R9.1
- net VIN+: now also C13.1, R15.2, R16.2; no longer C5.1, R11.2, R9.2
- net VS: now also R3.2; no longer R1.2
Other:
- moved on the sheet: C1, C10, C13, C14, C15, C2, C3, C5, C6, C7, C8, C9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

Commit message: Generated gerbers for Mrk 0.1
Added Gerbers for Mrk 0.1 revision, fixed silk screen issues, added pullup resistors for on board I2C on shortwave module, and changed amplifiers on longwave module (eliminated use of LTC2054HV, and switched to using LTC2050HV due to availability), also fixed (flipped) thermistor arraignment on shortwave module
Parts:
- JP1: value JUMPER-SMT_2_NC_PASTE_SILK -> JUMPER-SMT_2_NO_SILK; device SparkFun-Jumpers:JUMPER-SMT_2_NC_PASTE_SILK -> SparkFun-Jumpers:JUMPER-SMT_2_NO_SILK
- U3, U4: value LTC2050 -> LTC2054; device bschulz:LTC2050 -> bschulz:LTC2054
Changed lines of the file:
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@@
 <grid distance="0.1" unitdist="inch" unit="inch" style="lines" multiple="1" display="no" altdistance="0.01" altunitdist="inch" altunit="inch"/>
 <layers>
-<layer number="1" name="Top" color="4" fill="1" visible="yes" active="no"/>
-<layer number="2" name="Route2" color="1" fill="3" visible="yes" active="no"/>
-<layer number="3" name="Route3" color="4" fill="3" visible="yes" active="no"/>
-<layer number="4" name="Route4" color="1" fill="4" visible="yes" active="no"/>
-<layer number="5" name="Route5" color="4" fill="4" visible="yes" active="no"/>
-<layer number="6" name="Route6" color="1" fill="8" visible="yes" active="no"/>
-<layer number="7" name="Route7" color="4" fill="8" visible="yes" active="no"/>
-<layer number="8" name="Route8" color="1" fill="2" visible="yes" active="no"/>
-<layer number="9" name="Route9" color="4" fill="2" visible="yes" active="no"/>
-<layer number="10" name="Route10" color="1" fill="7" visible="yes" active="no"/>
-<layer number="11" name="Route11" color="4" fill="7" visible="yes" active="no"/>
-<layer number="12" name="Route12" color="1" fill="5" visible="yes" active="no"/>
-<layer number="13" name="Route13" color="4" fill="5" visible="yes" active="no"/>
-<layer number="14" name="Route14" color="1" fill="6" visible="yes" active="no"/>
-<layer number="15" name="Route15" color="4" fill="6" visible="yes" active="no"/>
-<layer number="16" name="Bottom" color="1" fill="1" visible="yes" active="no"/>
-<layer number="17" name="Pads" color="2" fill="1" visible="yes" active="no"/>
-<layer number="18" name="Vias" color="2" fill="1" visible="yes" active="no"/>
-<layer number="19" name="Unrouted" color="6" fill="1" visible="yes" active="no"/>
-<layer number="20" name="Dimension" color="24" fill="1" visible="yes" active="no"/>
-<layer number="21" name="tPlace" color="7" fill="1" visible="yes" active="no"/>
-<layer number="22" name="bPlace" color="7" fill="1" visible="yes" active="no"/>
-<layer number="23" name="tOrigins" color="15" fill="1" visible="yes" active="no"/>
-<layer number="24" name="bOrigins" color="15" fill="1" visible="yes" active="no"/>
-<layer number="25" name="tNames" color="7" fill="1" visible="yes" active="no"/>
-<layer number="26" name="bNames" color="7" fill="1" visible="yes" active="no"/>
-<layer number="27" name="tValues" color="7" fill="1" visible="yes" active="no"/>
-<layer number="28" name="bValues" color="7" fill="1" visible="yes" active="no"/>
+<layer number="1" name="Top" color="4" fill="1" visible="no" active="no"/>
+<layer number="2" name="Route2" color="1" fill="3" visible="no" active="no"/>
+<layer number="3" name="Route3" color="4" fill="3" visible="no" active="no"/>
+<layer number="4" name="Route4" color="1" fill="4" visible="no" active="no"/>
+<layer number="5" name="Route5" color="4" fill="4" visible="no" active="no"/>
+<layer number="6" name="Route6" color="1" fill="8" visible="no" active="no"/>
+<layer number="7" name="Route7" color="4" fill="8" visible="no" active="no"/>
+<layer number="8" name="Route8" color="1" fill="2" visible="no" active="no"/>
+<layer number="9" name="Route9" color="4" fill="2" visible="no" active="no"/>
+<layer number="10" name="Route10" color="1" fill="7" visible="no" active="no"/>
+<layer number="11" name="Route11" color="4" fill="7" visible="no" active="no"/>
+<layer number="12" name="Route12" color="1" fill="5" visible="no" active="no"/>
+<layer number="13" name="Route13" color="4" fill="5" visible="no" active="no"/>
+<layer number="14" name="Route14" color="1" fill="6" visible="no" active="no"/>
+<layer number="15" name="Route15" color="4" fill="6" visible="no" active="no"/>
+<layer number="16" name="Bottom" color="1" fill="1" visible="no" active="no"/>
+<layer number="17" name="Pads" color="2" fill="1" visible="no" active="no"/>
+<layer number="18" name="Vias" color="2" fill="1" visible="no" active="no"/>
+<layer number="19" name="Unrouted" color="6" fill="1" visible="no" active="no"/>
+<layer number="20" name="Dimension" color="24" fill="1" visible="no" active="no"/>
+<layer number="21" name="tPlace" color="7" fill="1" visible="no" active="no"/>
+<layer number="22" name="bPlace" color="7" fill="1" visible="no" active="no"/>
+<layer number="23" name="tOrigins" color="15" fill="1" visible="no" active="no"/>
+<layer number="24" name="bOrigins" color="15" fill="1" visible="no" active="no"/>
+<layer number="25" name="tNames" color="7" fill="1" visible="no" active="no"/>
+<layer number="26" name="bNames" color="7" fill="1" visible="no" active="no"/>
+<layer number="27" name="tValues" color="7" fill="1" visible="no" active="no"/>
+<layer number="28" name="bValues" color="7" fill="1" visible="no" active="no"/>
 <layer number="29" name="tStop" color="7" fill="3" visible="no" active="no"/>
 <layer number="30" name="bStop" color="7" fill="6" visible="no" active="no"/>
@@
 <layer number="35" name="tGlue" color="7" fill="4" visible="no" active="no"/>
 <layer number="36" name="bGlue" color="7" fill="5" visible="no" active="no"/>
-<layer number="37" name="tTest" color="7" fill="1" visible="yes" active="no"/>
-<layer number="38" name="bTest" color="7" fill="1" visible="yes" active="no"/>
+<layer number="37" name="tTest" color="7" fill="1" visible="no" active="no"/>
+<layer number="38" name="bTest" color="7" fill="1" visible="no" active="no"/>
 <layer number="39" name="tKeepout" color="4" fill="11" visible="no" active="no"/>
 <layer number="40" name="bKeepout" color="1" fill="11" visible="no" active="no"/>
@@
 <layer number="44" name="Drills" color="7" fill="1" visible="no" active="no"/>
 <layer number="45" name="Holes" color="7" fill="1" visible="no" active="no"/>
-<layer number="46" name="Milling" color="3" fill="1" visible="yes" active="no"/>
-<layer number="47" name="Measures" color="7" fill="1" visible="yes" active="no"/>
-<layer number="48" name="Document" color="7" fill="1" visible="yes" active="no"/>
-<layer number="49" name="Reference" color="7" fill="1" visible="yes" active="no"/>
-<layer number="50" name="dxf" color="7" fill="1" visible="yes" active="no"/>
-<layer number="51" name="tDocu" color="7" fill="1" visible="yes" active="no"/>
-<layer number="52" name="bDocu" color="7" fill="1" visible="yes" active="no"/>
-<layer number="53" name="tGND_GNDA" color="7" fill="1" visible="yes" active="no"/>
-<layer number="54" name="bGND_GNDA" color="7" fill="1" visible="yes" active="no"/>
-<layer number="56" name="wert" color="7" fill="1" visible="yes" active="no"/>
-<layer number="57" name="tCAD" color="7" fill="1" visible="yes" active="no"/>
-<layer number="59" name="tCarbon" color="7" fill="1" visible="yes" active="no"/>
-<layer number="60" name="bCarbon" color="7" fill="1" visible="yes" active="no"/>
+<layer number="46" name="Milling" color="3" fill="1" visible="no" active="no"/>
+<layer number="47" name="Measures" color="7" fill="1" visible="no" active="no"/>
+<layer number="48" name="Document" color="7" fill="1" visible="no" active="no"/>
+<layer number="49" name="Reference" color="7" fill="1" visible="no" active="no"/>
+<layer number="50" name="dxf" color="7" fill="1" visible="no" active="no"/>
+<layer number="51" name="tDocu" color="7" fill="1" visible="no" active="no"/>
+<layer number="52" name="bDocu" color="7" fill="1" visible="no" active="no"/>
+<layer number="53" name="tGND_GNDA" color="7" fill="1" visible="no" active="no"/>
+<layer number="54" name="bGND_GNDA" color="7" fill="1" visible="no" active="no"/>
+<layer number="56" name="wert" color="7" fill="1" visible="no" active="no"/>
+<layer number="57" name="tCAD" color="7" fill="1" visible="no" active="no"/>
+<layer number="59" name="tCarbon" color="7" fill="1" visible="no" active="no"/>
+<layer number="60" name="bCarbon" color="7" fill="1" visible="no" active="no"/>
 <layer number="88" name="SimResults" color="9" fill="1" visible="yes" active="yes"/>
 <layer number="89" name="SimProbes" color="9" fill="1" visible="yes" active="yes"/>
@@
 <part name="D2" library="bschulz" deviceset="PHOTODIODE" device="VEMD1060" value="PHOTODIODEVEMD1060"/>
 <part name="D1" library="bschulz" deviceset="PHOTODIODE" device="SD003-151-001"/>
-<part name="U3" library="bschulz" deviceset="LTC2050" device="" value="LTC2050"/>
-<part name="U4" library="bschulz" deviceset="LTC2050" device="" value="LTC2050"/>
+<part name="U3" library="bschulz" deviceset="LTC2054" device="" value="LTC2054"/>
+<part name="U4" library="bschulz" deviceset="LTC2054" device="" value="LTC2054"/>
 <part name="R2" library="bschulz_passives" deviceset="R-EU_" device="R0603" technology="P1K" value="1k"/>
 <part name="C3" library="bschulz_passives" deviceset="C-EU" device="C0603" technology="0.15UF" value="0.15uF"/>
@@
 <part name="J3" library="bschulz" deviceset="CONN_4" device="2.54"/>
 <part name="J4" library="bschulz" deviceset="CONN_4" device="2.54"/>
-<part name="JP1" library="SparkFun-Jumpers" library_urn="urn:adsk.eagle:library:528" deviceset="JUMPER-SMT_2_NC_PASTE" device="_SILK" package3d_urn="urn:adsk.eagle:package:39282/1"/>
+<part name="JP1" library="SparkFun-Jumpers" library_urn="urn:adsk.eagle:library:528" deviceset="JUMPER-SMT_2_NO" device="_SILK" package3d_urn="urn:adsk.eagle:package:39279/1"/>
 <part name="GND5" library="supply1" library_urn="urn:adsk.eagle:library:371" deviceset="GND" device=""/>
 <part name="U1" library="bschulz" deviceset="ADXL343" device=""/>
