File: Hardware/Libelle_SmallBoard.brd (EAGLE design)
At the start: 36.8 x 31.8 mm, 56 parts, among them J1 CONN_42.54_SCREW, J2 CONN_42.54, J3 CONN_42.54, J4 CONN_42.54, Q1 2N7002, Q2 2N7002, Q3 DMG3404, U1 ADXL343, U2 ATTINY441/841841, U3 LTC2054, U4 LTC2054, U5 ADS1115, U6 TPS79733, U7 VEML6030, U8 VEML6075

Commit message: Add CITATION.cff; fix embedded project names in Eagle files
Co-Authored-By: Claude Sonnet 4.6 <noreply@anthropic.com>
Other:
- board text added: "Project Libelle v0.1 ShortWave ---------------- Developed by Northern Widget and University of Minnesota"
- board text removed: "Project Monarch v0.1 ShortWave ---------------- Developed by Northern Widget and University of Minnesota"
Changed lines of the file:
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@@
 <text x="22.225" y="30.48" size="0.8128" layer="52" font="vector" ratio="15" rot="MR90" align="center">SCL</text>
 <text x="18.415" y="6.731" size="0.8128" layer="52" font="vector" ratio="15" rot="MR0" align="center">3.3v ~ 5v</text>
-<text x="21.336" y="16.891" size="0.8128" layer="52" font="vector" ratio="15" rot="MR0" align="center-left">Project Monarch v0.1
+<text x="21.336" y="16.891" size="0.8128" layer="52" font="vector" ratio="15" rot="MR0" align="center-left">Project Libelle v0.1
 ShortWave
 ----------------
